File: RTC.kicad_sch (KiCad schematic)
At the start: 51 parts, among them J1 Conn_01x01_Socket, J2 Conn_01x01_Socket, X1 Power, X2 Address, X3 Data, X4 Mode, X5 Control, X6 Clock

Commit message: Add files via upload
Changed chip power-up reset schemtic, added IRQ option, fix silk problem.

Изменена схема сброса часов при подаче питания, добавлена опция IRQ, исправлены проблемы с шелкографией.
Parts:
- removed J1, J2: Conn_01x01_Socket, TestPoint:TestPoint_THTPad_D2.5mm_Drill1.2mm, symbol Connector:Conn_01x01_Socket
- added C2: 6n8, Capacitor_SMD:C_0805_2012Metric_Pad1.18x1.45mm_HandSolder, symbol Device:C
- added JP10: IRQ1, Jumper:SolderJumper-2_P1.3mm_Open_RoundedPad1.0x1.5mm, symbol Jumper:Jumper_2_Open
- added JP11: IRQ2, Jumper:SolderJumper-2_P1.3mm_Open_RoundedPad1.0x1.5mm, symbol Jumper:Jumper_2_Open
- added JP12: IRQ3, Jumper:SolderJumper-2_P1.3mm_Open_RoundedPad1.0x1.5mm, symbol Jumper:Jumper_2_Open
- added JP13: IRQ4, Jumper:SolderJumper-2_P1.3mm_Open_RoundedPad1.0x1.5mm, symbol Jumper:Jumper_2_Open
- added JP14: IRQ5, Jumper:SolderJumper-2_P1.3mm_Open_RoundedPad1.0x1.5mm, symbol Jumper:Jumper_2_Open
- added JP15: IRQ6, Jumper:SolderJumper-2_P1.3mm_Open_RoundedPad1.0x1.5mm, symbol Jumper:Jumper_2_Open
- added JP16: IRQ7, Jumper:SolderJumper-2_P1.3mm_Open_RoundedPad1.0x1.5mm, symbol Jumper:Jumper_2_Open
- added JP9: IRQ0, Jumper:SolderJumper-2_P1.3mm_Open_RoundedPad1.0x1.5mm, symbol Jumper:Jumper_2_Open
- added R1: 1k, Resistor_SMD:R_0805_2012Metric_Pad1.20x1.40mm_HandSolder, symbol Device:R
- added R3: 20k, Resistor_SMD:R_0805_2012Metric_Pad1.20x1.40mm_HandSolder, symbol Device:R
- added X7: Conn_01x10, Connector_PinHeader_2.54mm:PinHeader_1x10_P2.54mm_Vertical, symbol Connector_Generic:Conn_01x10
- BT1: footprint Battery:BatteryHolder_MYOUNG_BS-07-A1BJ001_CR2032 -> Battery:BatteryHolder_Keystone_500
- D1: renamed from D2; footprint Diode_SMD:D_SOD-123 -> Diode_SMD:D_SOD-123F
- R4: renamed from R2; value 22M -> 10M
- renumbered C11 to C1, C17 to C10, C1 to C11, C3 to C12, C7 to C13, C12 to C14, C2 to C15, C4 to C16, C8 to C17, C13 to C18, C5 to C3, C14 to C4, C15 to C5, C9 to C7, C10 to C8, C16 to C9, D1 to D2, DD5 to DD2, DD6 to DD3, DD2 to DD5, DD3 to DD6, R3 to R2, R1 to R5, R4 to R6, R5 to R7
Connections:
- net +5: now also R1.2
- net GND: now also DD5.11, C2.2, X7.1 (Pin_1), X7.10 (Pin_10); no longer DD1.1, DD1.2
- net RESOUT: no longer DD5.11
- net IRQ_RTC: now reaches DD1.3
- net IRQ_RTC: now also JP10.1 (A), JP11.1 (A), JP12.1 (A), JP13.1 (A), JP14.1 (A), JP15.1 (A), JP16.1 (A), JP9.1 (A)
- net at C7.1, C8.1, D1.1 (K)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: now also R3.1
- net at DD2.19 (~{IRQ}): now also DD1.1, DD1.2, R1.1
- net ~{RTC_RESET}: no longer names the net of DD2.18 (~{RST})
- net ~{RTC_RESET}: now also C2.1, R3.2; no longer DD5.10
- new net IRQ0: JP9.2 (B), X7.9 (Pin_9)
- new net IRQ1: JP10.2 (B), X7.8 (Pin_8)
- new net IRQ2: JP11.2 (B), X7.7 (Pin_7)
- new net IRQ3: JP12.2 (B), X7.6 (Pin_6)
- new net IRQ4: JP13.2 (B), X7.5 (Pin_5)
- new net IRQ5: JP14.2 (B), X7.4 (Pin_4)
- new net IRQ6: JP15.2 (B), X7.3 (Pin_3)
- new net IRQ7: JP16.2 (B), X7.2 (Pin_2)
- no-connect marks 8 -> 6
Other:
- title: Модуль часов реального времени -> Модуль часов\n реального времени
- moved on the sheet: BT1, C1, D1, D2, D3, DD1A, DD5E, JP1, R2, R6

Commit message: Add files via upload
Fix start-up reset issue

Устранение проблемы начального сброса
Parts:
- C2: value 6n8 -> 4n7
Connections:
- net +5: now also R3.1
- net at C7.1, C8.1, D1.1 (K)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: no longer R3.1
Changed lines of the file:
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@@
 	(title_block
 		(title "Модуль часов\\n реального времени")
-		(date "2026-02-19")
+		(date "2026-03-11")
 		(company "R2AKT")
 		(comment 1 "R2AKT.467863.001")
@@
 		(color 0 0 0 0)
 	)
-	(junction
-		(at 186.944 84.582)
-		(diameter 0)
-		(color 0 0 0 0)
-	)
 	(no_connect
 		(at 52.07 268.224)
@@
 	(wire
 		(pts
+			(xy 186.944 90.678) (xy 212.09 90.678)
+		)
+		(stroke
+			(width 0)
+			(type default)
+		)
+	)
+	(wire
+		(pts
 			(xy 395.478 39.878) (xy 394.208 39.878)
 		)
@@
 	(wire
 		(pts
-			(xy 286.512 156.972) (xy 289.052 156.972)
+			(xy 212.09 90.678) (xy 212.09 93.218)
 		)
 		(stroke
@@
 	(wire
 		(pts
-			(xy 127 153.162) (xy 127 167.132)
+			(xy 286.512 156.972) (xy 289.052 156.972)
 		)
 		(stroke
@@
 	(wire
 		(pts
-			(xy 186.944 83.058) (xy 186.944 84.582)
+			(xy 127 153.162) (xy 127 167.132)
 		)
 		(stroke
@@
 	(wire
 		(pts
+			(xy 186.944 83.058) (xy 186.944 90.678)
+		)
+		(stroke
+			(width 0)
+			(type default)
+		)
+	)
+	(wire
+		(pts
 			(xy 127 179.832) (xy 127 167.132)
 		)
@@
 	(wire
 		(pts
-			(xy 177.292 84.582) (xy 186.944 84.582)
+			(xy 177.292 84.582) (xy 205.232 84.582)
 		)
 		(stroke
@@
 		)
 	)
-	(wire
-		(pts
-			(xy 186.944 84.582) (xy 205.232 84.582)
-		)
-		(stroke
-			(width 0)
-			(type default)
-		)
-	)
 	(bus
 		(pts
@@
 			)
 		)
-		(property "Value" "6n8"
+		(property "Value" "4n7"
 			(at 193.548 69.342 90)
 			(effects

Commit message: Add files via upload
Parts:
- added C9: 100n, Capacitor_SMD:C_0805_2012Metric_Pad1.18x1.45mm_HandSolder, symbol Device:C
- added D1, D2, D4: 1N4148WS, Diode_SMD:D_SOD-323_HandSoldering, symbol Diode:1N4148WS
- added JP1: Btr. PWR, Jumper:SolderJumper-2_P1.3mm_Open_RoundedPad1.0x1.5mm, symbol Jumper:Jumper_2_Open
- added R4: 1k, Resistor_SMD:R_0805_2012Metric_Pad1.20x1.40mm_HandSolder, symbol Device:R
- added X8: RTC Standby, Connector_PinHeader_2.54mm:PinHeader_1x02_P2.54mm_Vertical, symbol Connector_Generic:Conn_01x02
- C1, C2: value 4n7 -> 6n8
- D6: renamed from D3; footprint Diode_SMD:D_SOD-323 -> Diode_SMD:D_SOD-323_HandSoldering
- R2: value 20k -> 10k
- R3: value 20k -> 1k
- renumbered C9 to C10, C10 to C11, C11 to C12, C12 to C13, C13 to C14, C14 to C15, C15 to C16, C16 to C17, C17 to C18, C18 to C19, D1 to D3, D2 to D5, JP9 to JP10, JP10 to JP11, JP11 to JP12, JP12 to JP13, JP13 to JP14, JP14 to JP15, JP15 to JP16, JP16 to JP17, JP1 to JP2, JP2 to JP3, JP3 to JP4, JP4 to JP5, JP5 to JP6, JP6 to JP7, JP7 to JP8, JP8 to JP9, R4 to R5, R5 to R6, R6 to R7, R7 to R8
Connections:
- net +5: now also D2.1 (K)
- net GND: now also C9.2, X8.1 (Pin_1)
- net at BT1.1 (+), D3.2 (A): now also JP2.2 (B), D4.1 (K); no longer JP2.1 (A)
- net at DD3.3 (Ia=b), R8.1: now also C9.1
- net at R7.2: now also JP2.1 (A); no longer JP2.2 (B)
- net at C7.1, C8.1, D3.1 (K)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: now also D1.1 (K)
- net at C2.1, DD2.18 (~{RST}), R3.2: now also D2.2 (A)
- net at C1.1, DD2.22 (PS), R2.2: now also D1.2 (A)
- net INTE renamed ~{WRQ}
- net Single_BCLK renamed F2TTL
- net Single_OSC_TTL renamed OSC_TTL
- new net: JP1.1 (A), R4.2
- new net: D4.2 (A), R4.1
- new net +5VSB: JP1.2 (B), X8.2 (Pin_2)
- no-connect marks 6 -> 7
Other:
- moved on the sheet: BT1, C1, C2, C7, C8, D3, D5, D6, DD1A, DD4B, DD4D, DD5A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
